File: RAMs/RAM_TheoreticalDiagram.sch (EAGLE design)
At the start: 20 parts, among them IC1 74HC573D, IC10 74HC573D, IC11 74HC573D, IC12 74HC573D, IC13 74HC573D, IC14 74HC573D, IC15 74HC573D, IC16 74HC573D, IC17 74HC154DW, IC18 74HC154DW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

Commit message: Finished the Read/Write Verification
Parts:
- added IC21, IC22, IC23: 4049D, 40xx:4049D
Connections:
- new net N$47: IC17A.0, IC21A.I
- new net N$52: IC17A.1, IC21B.I
- new net N$53: IC17A.2, IC21C.I
- new net N$54: IC17A.3, IC21D.I
- new net N$55: IC17A.4, IC21E.I
- new net N$56: IC17A.5, IC21F.I
- new net N$58: IC17A.6, IC22A.I
- new net N$59: IC17A.7, IC22B.I
- new net N$60: IC17A.8, IC22C.I
- new net N$61: IC17A.9, IC22D.I
- new net N$62: IC17A.10, IC22E.I
- new net N$64: IC17A.11, IC22F.I
- new net N$66: IC17A.12, IC23A.I
- new net N$67: IC17A.13, IC23B.I
- new net N$68: IC17A.14, IC23C.I
- new net N$69: IC17A.15, IC23D.I
- new net N$72: IC19A.O, IC23E.I
- new net N$73: IC19B.O, IC23F.I
- net N$1: now also IC23A.O; no longer IC17A.12
- net N$14: now also IC22E.O; no longer IC17A.10
- net N$15: now also IC22D.O; no longer IC17A.9
- net N$18: now also IC22F.O; no longer IC17A.11
- net N$22: now also IC21E.O; no longer IC17A.4
- net N$23: now also IC21F.O; no longer IC17A.5
- net N$29: now also IC22A.O; no longer IC17A.6
- net N$3: now also IC23B.O; no longer IC17A.13
- net N$31: now also IC22B.O; no longer IC17A.7
- net N$34: now also IC21A.O; no longer IC17A.0
- net N$36: now also IC21B.O; no longer IC17A.1
- net N$38: now also IC21C.O; no longer IC17A.2
- net N$40: now also IC21D.O; no longer IC17A.3
- net N$42: now also IC23F.O; no longer IC19A.O
- net N$43: now also IC23E.O; no longer IC19B.O
- net N$5: now also IC23C.O; no longer IC17A.14
- net N$7: now also IC23D.O; no longer IC17A.15
- net N$9: now also IC22C.O; no longer IC17A.8
Other:
- note added: "DATA I/O"
- note removed: "DATA INPUT"
- note removed: "DATA OUTPUT"
- moved on the sheet: IC17, IC19A, IC19B, IC20A
